Commit message: Remove left files

File: robot_frame/description/ladle.xacro (robot description, xacro)
@@ -104,3 +104,44 @@
         </xacro:plate_panel>
     </link>
+    <!-- JOINTS -->
+    <!-- JOINT: LADLE BRACKET + BRACKET HOLDER LEFT -->
+    <joint name="ladle_lbr_holder_joint" type="revolute">
+        <parent link="box_bracket_holder_left"/>
+        <child link="ladle_bracket_horizontal"/>
+        <axis xyz="0 1 0"/>
+        <origin xyz="0 -${box_bracket_ladle_width/2 - box_bracket_holder_depth/2} 0" rpy="0 0 0" />
+        <limit effort="500.0" lower="-0.48" upper="0.4" velocity=".5"/>
+    </joint>
+    <!-- JOINT: LADLE BRACKET VERTICAL LEFT + LADLE BRACKET (HORIZONTAL) -->
+    <joint name="vbracket_hbracket_left_joint" type="fixed">
+        <parent link="ladle_bracket_horizontal"/>
+        <child link="ladle_bracket_vertical_left"/>
+        <origin xyz="${ladle_bracket_vertical_depth/2} ${ladle_bracket_length/3} 0" />
+    </joint>
+    <!-- JOINT: LADLE BRACKET VERTICAL RIGHT + LADLE BRACKET (HORIZONTAL) -->
+    <joint name="vbracket_hbracket_joint_right" type="fixed">
+        <parent link="ladle_bracket_horizontal"/>
+        <child link="ladle_bracket_vertical_right"/>
+        <origin xyz="${ladle_bracket_vertical_depth/2} -${ladle_bracket_length/3} 0" />
+    </joint>
+    <!-- JOINT: LADLE BRACKET (HORIZONTAL) + STEEVE -->
+    <joint name="steeve_vbracket_joint" type="revolute">
+        <parent link="ladle_bracket_vertical_left"/>
+        <child link="ladle_steeve"/>
+        <axis xyz="0 1 0"/>
+        <origin xyz="${ladle_bracket_vertical_depth/2} -${ladle_sleeve_length/4 - ladle_bracket_vertical_width/2} 0" />
+        <limit effort="100.0" lower="-1.3" upper="0.3" velocity="1.0"/>
+    </joint>
+    <!-- JOINT: LADLE STEEVE + LADLE PLATE TOP -->
+    <joint name="tplate_steeve_joint" type="fixed">
+        <parent link="ladle_steeve"/>
+        <child link="ladle_plate_top"/>
+        <origin xyz="${ladle_plate_depth + ladle_sleeve_radius/2} 0 ${ladle_plate_height/2 - ladle_sleeve_radius}" rpy="0 0 0" />
+    </joint>
+    <!-- JOINT: LADLE PLATE TOP + LADLE PLATE BOTTOM -->
+    <joint name="bplate_tplate_joint" type="fixed">
+        <parent link="ladle_plate_top"/>
+        <child link="ladle_plate_bottom"/>
+        <origin xyz="${ladle_plate_depth/2} 0 -${ladle_plate_height/2 + ladle_plate_depth}" />
+    </joint>
 </robot>

File: robot_frame/description/manipulators.xacro (robot description, xacro)
@@ -1,5 +1,5 @@
 <?xml version="1.0"?>
 <robot xmlns:xacro="http://www.ros.org/wiki/xacro">
-	<!-- DAE image of finger manipulator -->
+    <!-- DAE image of finger manipulator -->
     <xacro:macro name="finger" params="type:=''">
         <mesh filename="file://$(arg resDir)/gripper/l_finger_${type}.dae" scale="0.5 0.5 0.5"/>

File: robot_frame/description/robot.urdf.xacro (robot description, xacro)
@@ -18,9 +18,8 @@
     <xacro:include filename="manipulators.xacro"/>
     <xacro:include filename="manipulator_joints.xacro"/>
+    <!-- [UNUSED] -->
     <!-- LADLE AND JOINTS -->
-    <!-- [DEBUG] -->
     <!--
     <xacro:include filename="ladle.xacro"/>
-    <xacro:include filename="ladle_joints.xacro"/>
     -->
     <!-- BASIS LINK -->
@@ -117,5 +116,8 @@
         <origin xyz="${box_bracket_ladle_depth+ box_bracket_ladle_depth/2} -${box_bracket_ladle_width/2 - box_bracket_holder_width/2} 0"/>
     </joint>
-    <!-- LADLE (INCLUDES)-->
+    <!-- LADLE -->
+    <!-- -->
+    <!-- DESCRIPTION INCLUDES -->
+    <!-- -->
     <!-- BOX PANELS -->
     <!-- JOINT: PANEL BACK + CHASSIS -->
